Commit message: Added slidingModeControl

File: dd_bot/urdf/dd_bot.xacro (robot description, xacro)
@@ -108,5 +108,5 @@
       <origin xyz="0 0 0.0" rpy="0 0 0" />
       <geometry>
-          <cylinder length="0.02" radius="0.01" />
+          <cylinder length="0.04" radius="0.01" />
       </geometry>
       <material name="darkgray">
@@ -118,5 +118,5 @@
     <parent link = "base_link"/>
     <child link = "laser"/>
-    <origin xyz="0.04 0 0.05" rpy="0 0 0"/>
+    <origin xyz="0.04 0 0.06" rpy="0 0 0"/>
   </joint>
   <transmission name="left_wheel_tran">
